Commit message: add mesh file and mass properties

File: armsauv_description/robots/default.xacro (robot description, xacro)
@@ -3,14 +3,17 @@
   <xacro:arg name="debug" default="0"/>
   <xacro:arg name="namespace" default="armsauv"/>
+  <xacro:arg name="inertial_reference_frame" default="world"/>
   <!-- Include the ROV macro file -->
   <xacro:include filename="$(find armsauv_description)/urdf/base.xacro"/>
   <xacro:include filename="$(find armsauv_description)/urdf/gazebo.xacro"/>
   <!-- Create the armsauv -->
-  <xacro:armsauv_base namespace="$(arg namespace)">
+  <xacro:armsauv_base
+    namespace="$(arg namespace)"
+    inertial_reference_frame="$(arg inertial_reference_frame)">
     <!-- The underwater object plugin is given as an input block parameter to
      allow the addition of external models of manipulator units -->
     <gazebo>
       <plugin name="uuv_plugin" filename="libuuv_underwater_object_ros_plugin.so">
-        <fluid_density>1028.0</fluid_density>
+        <fluid_density>1025.0</fluid_density>
         <flow_velocity_topic>hydrodynamics/current_velocity</flow_velocity_topic>
         <debug>$(arg debug)</debug>

File: armsauv_description/urdf/actuators.xacro (robot description, xacro)
@@ -9,24 +9,24 @@
     -->
     <xacro:thruster_macro robot_namespace="${namespace}" thruster_id="0">
-        <origin xyz="0 0 0" rpy="0 0 ${pi}" />
-    </xacro:thruster_macro>
-    <xacro:thruster_macro robot_namespace="${namespace}" thruster_id="1">
-        <origin xyz="0 0 0" rpy="0 0 ${pi}" />
-    </xacro:thruster_macro>
-    <xacro:thruster_macro robot_namespace="${namespace}" thruster_id="2">
-    <origin xyz="0 0 0" rpy="0 -${0.5*pi} 0" />
+        <origin xyz="-1.842 0 0" rpy="0 0 0" />
     </xacro:thruster_macro>
     <!-- Instantiate fins, if necessary -->
-    <xacro:fin_macro namespace="${namespace}" fin_id="0">
-      <origin xyz="0 0 0" rpy="0 0 0" />
-    </xacro:fin_macro>
-    <xacro:fin_macro namespace="${namespace}" fin_id="1">
-      <origin xyz="0 0 0" rpy="0 0 0" />
-    </xacro:fin_macro>
-    <xacro:fin_macro namespace="${namespace}" fin_id="2">
-      <origin xyz="0 0 0" rpy="0 0 0" />
-    </xacro:fin_macro>
-    <xacro:fin_macro namespace="${namespace}" fin_id="3">
-      <origin xyz="0 0 0" rpy="0 0 0" />
-    </xacro:fin_macro>
+    <xacro:front_fin_macro namespace="${namespace}" fin_id="0" mesh_filename="${front_fin_mesh_file}">
+      <origin xyz="0.528 -0.201 0" rpy="${0.5 * pi} 0 0" />
+    </xacro:front_fin_macro>
+    <xacro:front_fin_macro namespace="${namespace}" fin_id="1" mesh_filename="${front_fin_mesh_file}">
+      <origin xyz="0.528 0.201 0" rpy="${1.5 * pi} 0 0" />
+    </xacro:front_fin_macro>
+    <xacro:aft_fin_macro namespace="${namespace}" fin_id="2" mesh_filename="${aft_fin_mesh_file}">
+      <origin xyz="-1.537 0.136 0" rpy="${0.5 * pi} 0 0" />
+    </xacro:aft_fin_macro>
+    <xacro:aft_fin_macro namespace="${namespace}" fin_id="3" mesh_filename="${aft_fin_mesh_file}">
+      <origin xyz="-1.537 0 0.136" rpy="${1 * pi} 0 0" />
+    </xacro:aft_fin_macro>
+    <xacro:aft_fin_macro namespace="${namespace}" fin_id="4" mesh_filename="${aft_fin_mesh_file}">
+      <origin xyz="-1.537 -0.136 0" rpy="${1.5 * pi} 0 0" />
+    </xacro:aft_fin_macro>
+    <xacro:aft_fin_macro namespace="${namespace}" fin_id="5" mesh_filename="${aft_fin_mesh_file}">
+      <origin xyz="-1.537 0 -0.136" rpy="${0 * pi} 0 0" />
+    </xacro:aft_fin_macro>
 </robot>

File: armsauv_description/urdf/base.xacro (robot description, xacro)
@@ -12,9 +12,9 @@
     Vehicle's parameters (remember to enter the model parameters below)
   -->
-  <xacro:property name="mass" value="0"/>
+  <xacro:property name="mass" value="831"/>
   <!-- Center of gravity -->
-  <xacro:property name="cog" value="0 0 0"/>
+  <xacro:property name="cog" value="0 0 0.0086"/>
   <!-- Fluid density -->
-  <xacro:property name="rho" value="1028"/>
+  <xacro:property name="rho" value="1025"/>
   <!--
     Visual mesh file for the vehicle, usually in DAE (Collada) format. Be sure to store the
@@ -23,11 +23,11 @@
     Open the meshes for the RexROV vehicle in Blender to see an example on the mesh placement.
   -->
-  <xacro:property name="visual_mesh_file" value="file://$(find armsauv_description)/meshes/vehicle.dae"/>
+  <xacro:property name="visual_mesh_file" value="file://$(find armsauv_description)/meshes/body.dae"/>
   <!-- Collision geometry mesh, usually in STL format (it is recommended to keep
   this geometry as simple as possible to improve the performance the physics engine
   regarding the computation of collision forces) -->
-  <xacro:property name="collision_mesh_file" value="file://$(find armsauv_description)/meshes/vehicle.stl"/>
+  <xacro:property name="collision_mesh_file" value="file://$(find armsauv_description)/meshes/body.dae"/>
   <!-- Vehicle macro -->
-  <xacro:macro name="armsauv_base" params="namespace *gazebo">
+  <xacro:macro name="armsauv_base" params="namespace *gazebo inertial_reference_frame">
       <!-- Rigid body description of the base link -->
       <link name="${namespace}/base_link">
@@ -39,10 +39,10 @@
           <mass value="${mass}" />
           <origin xyz="${cog}" rpy="0 0 0"/>
-          <inertia ixx="0" ixy="0" ixz="0"
-                   iyy="0" iyz="0"
-                   izz="0" />
+          <inertia ixx="0.82" ixy="0" ixz="0"
+                   iyy="30.14" iyz="0"
+                   izz="30.14" />
         </inertial>
         <visual>
-          <origin xyz="0 0 0" rpy="0 0 0"/>
+          <origin xyz="-0.5 0 0" rpy="0 0 0"/>
           <geometry>
             <mesh filename="${visual_mesh_file}" scale="1 1 1" />
@@ -50,5 +50,5 @@
         </visual>
         <collision>
-          <origin xyz="0 0 0" rpy="0 0 0"/>
+          <origin xyz="0 0 0" rpy="0 0 0"/>s
           <geometry>
             <mesh filename="${collision_mesh_file}" scale="1 1 1" />

File: armsauv_description/urdf/gazebo.xacro (robot description, xacro)
@@ -4,9 +4,10 @@
     <xacro:property name="armsauv_cob" value="0 0 0"/>
     <!-- Vehicle's actual volume (Gazebo cannot compute the volume out of the mesh) -->
-    <xacro:property name="armsauv_volume" value="0"/>
+    <xacro:property name="armsauv_volume" value="0.838"/>
     <!-- Describing the dimensions of the vehicle's bounding box -->
-    <xacro:property name="armsauv_length" value="0"/>
-    <xacro:property name="armsauv_width"  value="0"/>
-    <xacro:property name="armsauv_height" value="0"/>
+    <xacro:property name="armsauv_length" value="2.712"/>
+    <xacro:property name="armsauv_width"  value="0.935"/>
+    <xacro:property name="armsauv_radius"  value="0.120"/>
+    <xacro:property name="armsauv_height" value="0.484"/>
     <xacro:macro name="armsauv_hydro_model" params="namespace">
       <!-- List of hydrodynamic models this robot's links -->
@@ -26,21 +27,14 @@
         <!-- Center of buoyancy -->
         <center_of_buoyancy>${armsauv_cob}</center_of_buoyancy>
-        <!--
-        Choose one of the hydrodynamic models below, all are based on
-        Fossen's equation of motion for underwater vehicles
-        Reference:
-        [1] Fossen, Thor I. Handbook of marine craft hydrodynamics and motion
-            control. John Wiley & Sons, 2011.
-        -->
         <!-- 1) Fossen's equation of motion -->
         <hydrodynamic_model>
           <type>fossen</type>
           <added_mass>
-            0 0 0 0 0 0
-            0 0 0 0 0 0
-            0 0 0 0 0 0
-            0 0 0 0 0 0
-            0 0 0 0 0 0
-            0 0 0 0 0 0
+            1     0     0     0     0     0
+            0     16    0     0     0     0
+            0     0     16    0     0     0
+            0     0     0     0.005 0     0
+            0     0     0     0     1.3   0
+            0     0     0     0     0     1.3
           </added_mass>
           <!--
@@ -49,5 +43,10 @@
           -->
           <linear_damping>
-            0 0 0 0 0 0
+            -2.4  0     0     0     0     0
+            0     -23   0     0     0     11.5
+            0     0     -23   0     -11.5 0
+            0     0     0     -0.3  0     0
+            0     0     3.1   0     -9.7  0
+            0     -3.1  0     0     0     -9.7
           </linear_damping>
           <!--
@@ -65,31 +64,11 @@
           -->
           <quadratic_damping>
-            0 0 0 0 0 0
+            -2.4   0      0      0       0      0
+            0      -80    0      0       0      0.3
+            0      0      -80    0       -0.3   0
+            0      0      0      -0.0006 0      0
+            0      0      1.5    0       -9.1   0
+            0      -1.5   0      0       0      -9.1
           </quadratic_damping>
-          <!--
-            In case you want to model a simple surface vessel, you can use the
-            implementation of linear (small angle) theory for boxed shaped vessels
-            by providing the following parameters. If you omit the area of the
-            water level plane area, it will be calculated from the bounding box
-            parameters. Uncomment the lines below in case you are simulating a
-            surface vessel.
-            For more details on these parameters and the computation of buoyancy
-            for vessels using this theory, check:
-              [1] Lecture Notes  TTK 4190 Guidance and Control of Vehicles (T. I. Fossen)
-                  http://www.fossen.biz/wiley/Ch4.pdf
-              [2] Fossen, Thor I. Handbook of marine craft hydrodynamics and motion
-                  control. John Wiley & Sons, 2011.
-          -->
-          <!--
-          <metacentric_width>0.0</metacentric_width>
-          <metacentric_length>0.0</metacentric_length>
-          <submerged_height>0.0</submerged_height>
-          -->
-        </hydrodynamic_model>
-        <!-- 2) This computes the added-mass and damping parameters for a sphere
-        in the fluid with the given radius -->
-        <hydrodynamic_model>
-          <type>sphere</type>
-          <radius>0</radius>
         </hydrodynamic_model>
       </link>

File: armsauv_description/urdf/snippets.xacro (robot description, xacro)
@@ -1,7 +1,5 @@
 <?xml version="1.0"?>
 <robot xmlns:xacro="http://www.ros.org/wiki/xacro">
-  <!--                                                                      -->
   <!-- MACRO FOR THRUSTER UNITS  -->
-  <!--                                                                      -->
   <!-- Provide the propeller mesh in a separate file with the rotation axis
   over propeller's frame X-axis in DAE (Collada) or STL format.
@@ -51,10 +49,10 @@
         <gain>1</gain>
         <!-- Maximum allowed input value for the input signal for thruster unit -->
-        <clampMax>0</clampMax>
+        <clampMax>-3000</clampMax>
         <!-- Minimum allowed value for the input signal for thruster unit -->
-        <clampMin>0</clampMin>
+        <clampMin>3000</clampMin>
         <!-- Minimum and maximum thrust force output allowed -->
-        <thrustMin>0</thrustMin>
-        <thrustMax>0</thrustMax>
+        <thrustMin>-50</thrustMin>
+        <thrustMax>50</thrustMax>
         <!--
         Value from 0 to 1 to set the efficiency of the output thrust force
@@ -69,83 +67,11 @@
         -->
         <propeller_efficiency>1</propeller_efficiency>
-        <!--
-        Choose one of the propeller dynamics models below for your implementation
-        This will describe the dynamic model for the state variable of your thruster unit,
-        which can be, e.g., the angular velocity of the propeller.
-        -->
-        <!-- 1) Simple zero-order model -->
-        <dynamics>
-          <type>ZeroOrder</type>
-        </dynamics>
-        <!-- 2) First order model -->
         <dynamics>
           <type>FirstOrder</type>
-          <timeConstant>0.0</timeConstant>
+          <timeConstant>0.05</timeConstant>
         </dynamics>
-        <!-- 3) Yoerger's nonlinear dynamic model
-        For information on the model description:
-        [1] D. R. Yoerger, J. G. Cooke, and J.-J. E. Slotine, "The influence of
-            thruster dynamics on underwater vehicle behavior and their incorporation
-            into control system design," IEEE Journal of Oceanic Engineering, vol. 15,
-            no. 3, pp. 167-178, Jul. 1990.
-        -->
-        <dynamics>
-          <type>Yoerger</type>
-          <alpha>0.0</alpha>
-          <beta>0.0</beta>
-        </dynamics>
-        <!-- 4) Bessa's nonlinear dynamic model
-        For information on the model description:
-        [2] Bessa, Wallace Moreira, Max Suell Dutra, and Edwin Kreuzer. "Thruster
-            dynamics compensation for the positioning of underwater robotic vehicles
-            through a fuzzy sliding mode based approach." ABCM Symposium Series in
-            Mechatronics. Vol. 2. 2006.
-        -->
-        <dynamics>
-          <type>Bessa</type>
-          <Jmsp>0.0</Jmsp>
-          <Kv1>0.0</Kv1>
-          <Kv2>0.0</Kv2>
-          <Kt>0.0</Kt>
-          <Rm>0.0</Rm>
-        </dynamics>
-        <!--
-        Choose one of the model for the steady-state curve describing the
-        relationship between the state variable and the output thrust force
-        -->
-        <!-- 1) Basic curve
-        Input: x
-        Output: thrust
-        Function: thrust = rotorConstant * x * abs(x)
-        -->
         <conversion>
           <type>Basic</type>
-          <rotorConstant>0.0</rotorConstant>
-        </conversion>
-        <!-- 2) Dead-zone nonlinearity described in Bessa, 2006
-        Input: x
-        Output: thrust
-        Function:
-        thrust = rotorConstantL * (x * abs(x) - deltaL), if x * abs(x) <= deltaL
-        thrust = 0, if deltaL < x * abs(x) < deltaR
-        thrust = rotorConstantR * (x * abs(x) - deltaR), if x * abs(x) >= deltaL
-        -->
-        <conversion>
-          <type>Bessa</type>
-          <rotorConstantL>0.0</rotorConstantL>
-          <rotorConstantR>0.0</rotorConstantR>
-          <deltaL>0.0</deltaL>
-          <deltaR>0.0</deltaR>
-        </conversion>
-        <!-- 3) Linear interpolation
-        If you have access to the thruster's data sheet, for example,
-        you can enter samples of the curve's input and output values
-        and the thruster output will be found through linear interpolation
-        of the given samples.
-        -->
-        <conversion>
-          <type>LinearInterp</type>
-          <inputValues>0 1 2 3</inputValues>
-          <outputValues>0 1 2 3</outputValues>
+          <rotorConstant>0.0002</rotorConstant>
         </conversion>
       </plugin>
@@ -155,95 +81,89 @@
     </gazebo>
   </xacro:macro>
-  <!--                                                                      -->
   <!-- MACRO FOR FIN/RUDDER UNITS  -->
-  <!--                                                                      -->
-  <!--
-    This macro can be used to add fins to the body of the vehicle, the fins
-    should be initialized in the actuators.xacro file. If you vehicle has no
-    fins, you can erase the macro below.
-  -->
   <!-- A separate mesh for the fin should be stored in the meshes folder -->
-  <xacro:property name="fin_mesh_file" value="file://$(find armsauv_description)/meshes/fin.dae"/>
-  <!-- Fin joint limits  -->
-  <xacro:property name="fin_min_joint_limit" value="${0.0 * d2r}"/>
-  <xacro:property name="fin_max_joint_limit" value="${0.0 * d2r}"/>
-  <xacro:macro name="fin_macro" params="namespace fin_id *origin">
-      <joint name="${namespace}/fin${fin_id}_joint" type="revolute">
-          <limit effort="0" lower="${fin_min_joint_limit}" upper="${fin_max_joint_limit}" velocity="0"/>
-          <xacro:insert_block name="origin"/>
-          <axis xyz="0 0 1"/>
-          <parent link="${namespace}/base_link" />
-          <child link="${namespace}/fin${fin_id}" />
-      </joint>
-      <link name="${namespace}/fin${fin_id}">
-        <inertial>
-          <mass value="0.001" />
-          <origin xyz="0 0 0" rpy="0 0 0"/>
-          <inertia ixx="0.000000017" ixy="0.0" ixz="0.0"
-                 iyy="0.000000017" iyz="0.0"
-                 izz="0.000000017" />
-        </inertial>
-        <visual>
-          <origin xyz="0 0 0" rpy="0 0 0" />
-          <geometry>
-            <mesh filename="${fin_mesh_file}" scale="1 1 1"/>
-          </geometry>
-        </visual>
-      </link>
-      <gazebo>
-        <plugin name="${namespace}_fin${fin_id}_model" filename="libuuv_fin_ros_plugin.so">
-          <!--
-            First order dynamics model for the fin joint dynamics,
-            replace an appropriate time constant
-          -->
-          <dynamics>
-            <type>FirstOrder</type>
-            <timeConstant>0.0</timeConstant>
-          </dynamics>
-          <!--
-            Definition of the lift and drag model, choose ONE of the models
-            below according to the model you want to use.
-          -->
-          <!--
-            1) References for the two line lift and drag model:
-              [1] https://en.wikipedia.org/wiki/Lift_coefficient
-              [2] http://gazebosim.org/tutorials?tut=aerodynamics&cat=plugins
-          -->
-          <liftdrag>
-            <type>TwoLines</type>
-            <area>${replace here the value for the area of the fin's cross section}</area>
-            <fluid_density>0.0</fluid_density>
-            <a0>0.0</a0>
-            <alpha_stall>0.0</alpha_stall>
-            <cla>0.0</cla><!-- ^= 0.244 when using deg -->
-            <cla_stall>0.0</cla_stall>
-            <cda>0.0</cda>
-            <cda_stall>0.0</cda_stall>
-          </liftdrag>
-          <!--
-            2) Reference for the quadratic lift and drag model:
-              [1] Engelhardtsen, Oystein. 3D AUV Collision Avoidance.
-                  MS thesis. Institutt for teknisk kybernetikk, 2007.
-                  https://brage.bibsys.no/xmlui/handle/11250/259834
-          -->
-          <liftdrag>
-            <type>Quadratic</type>
-            <lift_constant>0.0</lift_constant>
-            <drag_constant>0.0</drag_constant>
-          </liftdrag>
-          <!--
-            Further parameters necessary for the lift and drag plugin
-          -->
-          <!-- Current velocity topic -->
-          <current_velocity_topic>/hydrodynamics/current_velocity</current_velocity_topic>
-          <!-- Name of the correspodent fin link and joint  -->
-          <link_name>${namespace}/fin${fin_id}</link_name>
-          <joint_name>${namespace}/fin${fin_id}_joint</joint_name>
-          <!-- Output topic to publish the current angle of the fin joint -->
-          <output_topic>${namespace}/fins/${fin_id}/output</output_topic>
-          <input_topic>${namespace}/fins/${fin_id}/input</input_topic>
-          <wrench_topic>${namespace}/fins/${fin_id}/wrench_topic</wrench_topic>
-        </plugin>
-      </gazebo>
+  <xacro:property name="front_fin_mesh_file" value="file://$(find armsauv_description)/meshes/front_fin.dae"/>
+  <xacro:property name="aft_fin_mesh_file" value="file://$(find armsauv_description)/meshes/aft_fin.dae"/>
+  <!-- Fin properties -->
+  <xacro:property name="fin_rho" value="1025"/>
+  <xacro:property name="front_fin_area" value="0.0064"/>
+  <xacro:property name="front_fin_lift_coefficient" value="3.0"/>
+  <xacro:property name="front_fin_drag_coefficient" value="1.98"/>
+  <xacro:macro name="front_fin_macro" params="namespace fin_id *origin mesh_filename">
+      <xacro:fin_quadratic_macro
+        namespace="${namespace}"
+        parent_link="${namespace}/base_link"
+        fin_id="${fin_id}"
+        min_joint_limit="${-90.0 * d2r}"
+        max_joint_limit="${90.0 * d2r}"
+        mesh_filename="${mesh_filename}"
+        fin_dynamics_time_constant="0.2"
+        lift_constant="${0.5 * fin_rho * front_fin_area * front_fin_lift_coefficient}"
+        drag_constant="${0.5 * fin_rho * front_fin_area * front_fin_drag_coefficient}"
+        current_velocity_topic="current_velocity">
+        <xacro:insert_block name="origin"/>
+      </xacro:fin_quadratic_macro>
   </xacro:macro>
+  <xacro:property name="aft_fin_area" value="0.0164"/>
+  <xacro:property name="aft_fin_lift_coefficient" value="3.0"/>
+  <xacro:property name="aft_fin_drag_coefficient" value="1.98"/>
+  <xacro:macro name="aft_fin_macro" params="namespace fin_id *origin mesh_filename">
+      <xacro:fin_quadratic_macro
+        namespace="${namespace}"
+        parent_link="${namespace}/base_link"
+        fin_id="${fin_id}"
+        min_joint_limit="${-90.0 * d2r}"
+        max_joint_limit="${90.0 * d2r}"
+        mesh_filename="${mesh_filename}"
+        fin_dynamics_time_constant="0.2"
+        lift_constant="${0.5 * fin_rho * aft_fin_area * aft_fin_lift_coefficient}"
+        drag_constant="${0.5 * fin_rho * aft_fin_area * aft_fin_drag_coefficient}"
+        current_velocity_topic="current_velocity">
+        <xacro:insert_block name="origin"/>
+      </xacro:fin_quadratic_macro>
+  </xacro:macro>
+  <!-- <xacro:macro name="fin_macro" params="namespace fin_id *origin mesh_filename">
+      <xacro:fin_two_lines_macro
+        namespace="${namespace}"
+        parent_link="${namespace}/base_link"
+        fin_id="${fin_id}"
+        min_joint_limit="${-80*d2r}"
+        max_joint_limit="${80*d2r}"
+        mesh_filename="${mesh_filename}"
+        fin_dynamics_time_constant="0.1"
+        fin_cross_section_area="${fin_area}"
+        current_velocity_topic="current_velocity"
+        fluid_density="1025.0"
+        a0="0.0"
+        alpha_stall="1.57"
+        cla="${0.5 * fin_rho * fin_area * fin_lift_coefficient}"
+        cla_stall="0.0"
+        cda="${0.5 * fin_rho * fin_area * fin_drag_coefficient}"
+        cda_stall="0">
+        <xacro:insert_block name="origin"/>
+      </xacro:fin_two_lines_macro>
+    </xacro:macro> -->
+    <!-- <xacro:macro name="fin_macro" params="namespace fin_id *origin mesh_filename">
+      <xacro:fin_two_lines_macro
+        namespace="${namespace}"
+        parent_link="${namespace}/base_link"
+        fin_id="${fin_id}"
+        min_joint_limit="${-80*d2r}"
+        max_joint_limit="${80*d2r}"
+        mesh_filename="${mesh_filename}"
+        fin_dynamics_time_constant="0.1"
+        fin_cross_section_area="${fin_area}"
+        current_velocity_topic="current_velocity"
+        fluid_density="1025.0"
+        a0="0.0"
+        alpha_stall="0.436332313"
+        cla="2.435070629"
+        cla_stall="0"
+        cda="0"
+        cda_stall="0">
+        <xacro:insert_block name="origin"/>
+      </xacro:fin_two_lines_macro>
+    </xacro:macro> -->
+    <!-- cla_stall="-1.929963096"
+        cda="1.101841914" -->
 </robot>
