Commit message: modify model

File: armsauv_description/urdf/gazebo.xacro (robot description, xacro)
@@ -35,5 +35,5 @@
             0       0    130.513    0  -16.488   0
             0       0       0    0.386    0      0
-            0       0       0   -16.488 61.8     0
+            0       0   -16.488     0   61.8     0
             0     4.895     0       0     0    67.48
           </added_mass>
@@ -65,8 +65,8 @@
           <quadratic_damping>
           -3.9     0      0      0     0      0
-            0    -131     0      0     0   -4.204
-            0      0    -131     0  23.016    0
+            0  -373.287   0      0     0   -4.204
+            0      0  -489.07    0  23.016    0
             0      0      0   -0.117   0      0
-            0      0   23.342    0 -353.4064  0
+            0      0   23.342    0 -353.406   0
             0   0.419     0      0     0  -227.024
           </quadratic_damping>

File: armsauv_description/urdf/sensors.xacro (robot description, xacro)
@@ -1,10 +1,4 @@
 <?xml version="1.0"?>
 <robot xmlns:xacro="http://www.ros.org/wiki/xacro">
-  <!--
-    Some examples of sensors that can be added to the vehicle frame.
-    Set the origin of the sensor frames correctly for your application
-    Look into the sensor macros in the package uuv_sensor_ros_plugins/urdf for
-    more examples or add you own custom sensor units.
-  -->
   <!-- Mount a GPS. -->
   <xacro:default_gps namespace="${namespace}" parent_link="${namespace}/base_link" />
@@ -14,28 +8,85 @@
     parent_link="${namespace}/base_link"
     inertial_reference_frame="${inertial_reference_frame}" />
+  <xacro:macro name="arms_forward_multibeam_p900" params="namespace parent_link *origin">
+    <xacro:multibeam_sonar
+      namespace="${namespace}"
+      suffix=""
+      parent_link="${parent_link}"
+      topic="sonar"
+      mass="0.001"
+      update_rate="15"
+      samples="512"
+      fov="1.5708"
+      range_min="1.0"
+      range_max="100.0"
+      range_stddev="0.027"
+      mesh="">
+      <inertia ixx="0.0" ixy="0.0" ixz="0.0" iyy="0.0" iyz="0.0" izz="0.0" />
+      <xacro:insert_block name="origin" />
+      <visual>
+        <geometry>
+          <mesh filename="file://$(find uuv_sensor_ros_plugins)/meshes/p900.dae" scale="1 1 1"/>
+        </geometry>
+      </visual>
+    </xacro:multibeam_sonar>
+  </xacro:macro>
   <!-- Forward-looking sonar sensor -->
-  <!-- <xacro:forward_multibeam_p900 namespace="${namespace}" parent_link="${namespace}/base_link">
+  <xacro:arms_forward_multibeam_p900 namespace="${namespace}" parent_link="${namespace}/base_link">
     <origin xyz="0 0 0" rpy="0 0 0"/>
-  </xacro:forward_multibeam_p900> -->
+  </xacro:arms_forward_multibeam_p900>
   <!-- DVL  -->
-  <!-- <xacro:default_dvl namespace="${namespace}" parent_link="${namespace}/base_link">
+  <xacro:default_dvl namespace="${namespace}" parent_link="${namespace}/base_link">
     <origin xyz="0 0 0" rpy="0 0 0"/>
-  </xacro:default_dvl> -->
-  <!-- RPT  -->
-  <!-- <xacro:default_rpt namespace="${namespace}" parent_link="${namespace}/base_link">
+  </xacro:default_dvl>
+  <xacro:macro name="arms_pressure" params="namespace parent_link *origin">
+    <xacro:pressure_plugin_macro
+      namespace="${namespace}"
+      suffix=""
+      parent_link="${parent_link}"
+      topic="pressure"
+      mass="0.001"
+      update_rate="10"
+      range="30000"
+      noise_sigma="3.0"
+      noise_amplitude="0.0"
+      estimateDepth="false"
+      standardPressure="101.325"
+      kPaPerM="9.80638">
+      <inertia ixx="0.0" ixy="0.0" ixz="0.0" iyy="0.0" iyz="0.0" izz="0.0" />
+      <xacro:insert_block name="origin" />
+    </xacro:pressure_plugin_macro>
+  </xacro:macro>
+  <!-- Pressure  -->
+  <xacro:arms_pressure namespace="${namespace}" parent_link="${namespace}/base_link">
     <origin xyz="0 0 0" rpy="0 0 0"/>
-  </xacro:default_rpt> -->
-  <!-- Pressure  -->
-  <!-- <xacro:default_pressure namespace="${namespace}" parent_link="${namespace}/base_link">
+  </xacro:arms_pressure>
+  <xacro:macro name="arms_imu" params="namespace parent_link *origin">
+    <!-- ADIS16448 IMU. -->
+    <xacro:imu_plugin_macro
+      namespace="${namespace}"
+      imu_suffix=""
+      parent_link="${parent_link}"
+      imu_topic="imu"
+      mass_imu_sensor="0.001"
+      gyroscope_noise_density="0.0003394"
+      gyroscope_random_walk="0.000038785"
+      gyroscope_bias_correlation_time="1000.0"
+      gyroscope_turn_on_bias_sigma="0.0087"
+      accelerometer_noise_density="0.004"
+      accelerometer_random_walk="0.006"
+      accelerometer_bias_correlation_time="300.0"
+      accelerometer_turn_on_bias_sigma="0.1960"
+      orientation_noise="0.01"
+      enable_local_ned_frame="false"
+      reference_frame="world"
+      update_rate="50">
+      <inertia ixx="0.0" ixy="0.0" ixz="0.0" iyy="0.0" iyz="0.0" izz="0.0" />
+      <xacro:insert_block name="origin" />
+    </xacro:imu_plugin_macro>
+  </xacro:macro>
+  <!-- IMU  -->
+  <xacro:arms_imu namespace="${namespace}" parent_link="${namespace}/base_link">
     <origin xyz="0 0 0" rpy="0 0 0"/>
-  </xacro:default_pressure> -->
-  <!-- IMU  -->
-  <xacro:default_imu namespace="${namespace}" parent_link="${namespace}/base_link">
-    <origin xyz="0 0 0" rpy="0 0 0"/>
-  </xacro:default_imu>
-  <!-- Mount a camera -->
-  <!-- <xacro:default_camera namespace="${namespace}" parent_link="${namespace}/base_link">
-    <origin xyz="0 0 0" rpy="0 0 0"/>
-  </xacro:default_camera> -->
+  </xacro:arms_imu>
   <!-- Mount the chemical concentration sensor -->
   <xacro:chemical_concentration_sensor_macro

File: armsauv_description/urdf/snippets.xacro (robot description, xacro)
@@ -88,5 +88,5 @@
   <xacro:property name="fin_rho" value="1025"/>
   <xacro:property name="front_fin_area" value="0.0127"/>
-  <xacro:property name="front_fin_lift_coefficient" value="22.4905"/>
+  <xacro:property name="front_fin_lift_coefficient" value="20.843"/>
   <xacro:property name="front_fin_drag_coefficient" value="1.98"/>
   <xacro:macro name="front_fin_macro" params="namespace fin_id *origin mesh_filename">
