Commit message: first try

File: armsauv_description/urdf/actuators.xacro (robot description, xacro)
@@ -9,24 +9,24 @@
     -->
     <xacro:thruster_macro robot_namespace="${namespace}" thruster_id="0">
-        <origin xyz="-1.842 0 0" rpy="0 0 0" />
+        <origin xyz="-3.8 0 0" rpy="0 0 0" />
     </xacro:thruster_macro>
     <!-- Instantiate fins, if necessary -->
-    <xacro:front_fin_macro namespace="${namespace}" fin_id="0" mesh_filename="${front_fin_mesh_file}">
-      <origin xyz="0.528 -0.201 0" rpy="${0.5 * pi} 0 0" />
-    </xacro:front_fin_macro>
-    <xacro:front_fin_macro namespace="${namespace}" fin_id="1" mesh_filename="${front_fin_mesh_file}">
-      <origin xyz="0.528 0.201 0" rpy="${1.5 * pi} 0 0" />
-    </xacro:front_fin_macro>
-    <xacro:aft_fin_macro namespace="${namespace}" fin_id="2" mesh_filename="${aft_fin_mesh_file}">
-      <origin xyz="-1.537 0.136 0" rpy="${0.5 * pi} 0 0" />
-    </xacro:aft_fin_macro>
-    <xacro:aft_fin_macro namespace="${namespace}" fin_id="3" mesh_filename="${aft_fin_mesh_file}">
-      <origin xyz="-1.537 0 0.136" rpy="${1 * pi} 0 0" />
-    </xacro:aft_fin_macro>
-    <xacro:aft_fin_macro namespace="${namespace}" fin_id="4" mesh_filename="${aft_fin_mesh_file}">
-      <origin xyz="-1.537 -0.136 0" rpy="${1.5 * pi} 0 0" />
-    </xacro:aft_fin_macro>
-    <xacro:aft_fin_macro namespace="${namespace}" fin_id="5" mesh_filename="${aft_fin_mesh_file}">
-      <origin xyz="-1.537 0 -0.136" rpy="${0 * pi} 0 0" />
-    </xacro:aft_fin_macro>
+    <xacro:fin_macro namespace="${namespace}" fin_id="0" mesh_filename="${front_fin_mesh_file}">
+      <origin xyz="1.865 -0.699 0.013" rpy="${0.5 * pi} 0 0" />
+    </xacro:fin_macro>
+    <xacro:fin_macro namespace="${namespace}" fin_id="1" mesh_filename="${front_fin_mesh_file}">
+      <origin xyz="1.865 0.699 -0.287" rpy="${1.5 * pi} 0 0" />
+    </xacro:fin_macro>
+    <xacro:fin_macro namespace="${namespace}" fin_id="2" mesh_filename="${aft_fin_mesh_file}">
+      <origin xyz="-3.369 0.621 -0.1896" rpy="${0.5 * pi} 0 0" />
+    </xacro:fin_macro>
+    <xacro:rouder_macro namespace="${namespace}" fin_id="3" mesh_filename="${aft_fin_mesh_file}">
+      <origin xyz="-3.369 0 0.443" rpy="${1 * pi} 0 0" />
+    </xacro:rouder_macro>
+    <xacro:fin_macro namespace="${namespace}" fin_id="4" mesh_filename="${aft_fin_mesh_file}">
+      <origin xyz="-3.369 -0.621 -0.0844" rpy="${1.5 * pi} 0 0" />
+    </xacro:fin_macro>
+    <xacro:rouder_macro namespace="${namespace}" fin_id="5" mesh_filename="${aft_fin_mesh_file}">
+      <origin xyz="-3.369 0 -0.443" rpy="${0 * pi} 0 0" />
+    </xacro:rouder_macro>
 </robot>

File: armsauv_description/urdf/base.xacro (robot description, xacro)
@@ -12,7 +12,7 @@
     Vehicle's parameters (remember to enter the model parameters below)
   -->
-  <xacro:property name="mass" value="${831 / 9.8}"/>
+  <xacro:property name="mass" value="4390"/>
   <!-- Center of gravity -->
-  <xacro:property name="cog" value="0 0 0.0086"/>
+  <xacro:property name="cog" value="0 0 0"/>
   <!-- Fluid density -->
   <xacro:property name="rho" value="1025"/>
@@ -39,7 +39,7 @@
           <mass value="${mass}" />
           <origin xyz="${cog}" rpy="0 0 0"/>
-          <inertia ixx="0.82" ixy="0" ixz="0"
-                   iyy="30.14" iyz="0"
-                   izz="30.14" />
+          <inertia ixx="1315" ixy="0" ixz="0"
+                   iyy="5900" iyz="0"
+                   izz="5057" />
         </inertial>
         <visual>

File: armsauv_description/urdf/gazebo.xacro (robot description, xacro)
@@ -2,12 +2,15 @@
 <robot xmlns:xacro="http://www.ros.org/wiki/xacro">
     <!-- Center of buoyancy -->
-    <xacro:property name="armsauv_cob" value="0 0 0"/>
+    <!-- <xacro:property name="armsauv_cob" value="0.086 0 -0.137"/> -->
+    <xacro:property name="armsauv_cob" value="0.086 0 -0.137"/>
     <!-- Vehicle's actual volume (Gazebo cannot compute the volume out of the mesh) -->
-    <xacro:property name="armsauv_volume" value="${838 / 9.8 / 1000}"/>
+    <!-- <xacro:property name="armsauv_volume" value="${4605 / 1025}"/> -->
+    <!-- <xacro:property name="armsauv_volume" value="${4539 / 1025}"/> -->
+    <xacro:property name="armsauv_volume" value="${4390 / 1025}"/>
     <!-- Describing the dimensions of the vehicle's bounding box -->
-    <xacro:property name="armsauv_length" value="2.712"/>
-    <xacro:property name="armsauv_width"  value="0.935"/>
-    <xacro:property name="armsauv_radius"  value="0.120"/>
-    <xacro:property name="armsauv_height" value="0.484"/>
+    <xacro:property name="armsauv_length" value="8.534"/>
+    <xacro:property name="armsauv_width"  value="2.0801"/>
+    <xacro:property name="armsauv_radius"  value="0.35795"/>
+    <xacro:property name="armsauv_height" value="1.4318"/>
     <xacro:macro name="armsauv_hydro_model" params="namespace">
       <!-- List of hydrodynamic models this robot's links -->
@@ -37,4 +40,34 @@
             0       0   -16.488     0  78.266    0
             0     4.895     0       0     0    67.489
+            <!-- 302.286     0         0          0          0           0
+            0       12996.067     0          0          0        3778.498
+            0           0     7198.801       0       -138.636       0
+            0           0         0       2435.827      0           0
+            0           0     -138.636        0       40597.109     0
+            0       3778.498      0           0         0        42452.977 -->
+            <!-- 302.286     0         0          0          0           0
+            0       12996.067     0          0          0           0
+            0           0     7198.801       0          0           0
+            0           0         0       2435.827      0           0
+            0           0         0          0       40597.109      0
+            0           0         0          0         0        42452.977 -->
+            <!-- 302.286     0        0          0          0          0
+            0       12996.067    0       1486.934      0        3778.498
+            0           0     7198.801      0      -138.636       0
+            0        1486.934    0      2435.827       0       -85.834
+            0           0    -138.636       0       40597.109     0
+            0        3778.498    0       -85.834       0        42452.977 -->
+            <!-- 30.2285     0         0          0         0           0
+            0       1299.6067     0      -148.6934     0      -377.8498
+            0           0     719.8802       0       13.8636       0
+            0       -148.6934     0       243.5827     0        8.5834
+            0           0     13.8636        0      4059.7109      0
+            0       -377.8498     0        8.5834      0       4245.2977 -->
+            <!-- 302.285     0         0          0         0           0
+            0       12996.067     0          0         0           0
+            0           0     7198.802       0         0           0
+            0           0         0       2435.827     0           0
+            0           0         0        0      40597.109        0
+            0           0         0          0         0       42452.977 -->
           </added_mass>
           <!--

File: armsauv_description/urdf/snippets.xacro (robot description, xacro)
@@ -49,10 +49,10 @@
         <gain>1</gain>
         <!-- Maximum allowed input value for the input signal for thruster unit -->
-        <clampMax>2300</clampMax>
+        <clampMax>1000</clampMax>
         <!-- Minimum allowed value for the input signal for thruster unit -->
-        <clampMin>-2300</clampMin>
+        <clampMin>-1000</clampMin>
         <!-- Minimum and maximum thrust force output allowed -->
-        <thrustMin>-125</thrustMin>
-        <thrustMax>125</thrustMax>
+        <thrustMin>-36373000</thrustMin>
+        <thrustMax>36373000</thrustMax>
         <!--
         Value from 0 to 1 to set the efficiency of the output thrust force
@@ -71,18 +71,7 @@
           <timeConstant>0.05</timeConstant>
         </dynamics>
-        <!-- <conversion>
+        <conversion>
           <type>Basic</type>
-          <rotorConstant>0.0002</rotorConstant>
-        </conversion>         -->
-        <!-- 3) Linear interpolation
-        If you have access to the thruster's data sheet, for example,
-        you can enter samples of the curve's input and output values
-        and the thruster output will be found through linear interpolation
-        of the given samples.
-        -->
-        <conversion>
-          <type>LinearInterp</type>
-          <inputValues>888 1500 1700 1900 2100 2300</inputValues>
-          <outputValues>0 55 70 88 105 125</outputValues>
+          <rotorConstant>36.374</rotorConstant>
         </conversion>
       </plugin>
@@ -98,8 +87,8 @@
   <!-- Fin properties -->
   <xacro:property name="fin_rho" value="1025"/>
-  <xacro:property name="front_fin_area" value="0.0127"/>
-  <xacro:property name="front_fin_lift_coefficient" value="20.843"/>
-  <xacro:property name="front_fin_drag_coefficient" value="1.98"/>
-  <xacro:macro name="front_fin_macro" params="namespace fin_id *origin mesh_filename">
+  <xacro:property name="fin_area" value="1"/>
+  <xacro:property name="fin_lift_coefficient" value="373.249"/>
+  <xacro:property name="fin_drag_coefficient" value="1.98"/>
+  <xacro:macro name="fin_macro" params="namespace fin_id *origin mesh_filename">
       <xacro:fin_quadratic_macro
         namespace="${namespace}"
@@ -110,14 +99,14 @@
         mesh_filename="${mesh_filename}"
         fin_dynamics_time_constant="0.2"
-        lift_constant="${0.5 * fin_rho * front_fin_area * front_fin_lift_coefficient}"
-        drag_constant="${0.5 * fin_rho * front_fin_area * front_fin_drag_coefficient}"
+        lift_constant="${0.5 * fin_rho * fin_area * fin_lift_coefficient}"
+        drag_constant="${0.5 * fin_rho * fin_area * fin_drag_coefficient}"
         current_velocity_topic="current_velocity">
         <xacro:insert_block name="origin"/>
       </xacro:fin_quadratic_macro>
   </xacro:macro>
-  <xacro:property name="aft_fin_area" value="0.0172"/>
-  <xacro:property name="aft_fin_lift_coefficient" value="19.1395"/>
-  <xacro:property name="aft_fin_drag_coefficient" value="1.98"/>
-  <xacro:macro name="aft_fin_macro" params="namespace fin_id *origin mesh_filename">
+  <xacro:property name="rouder_area" value="1"/>
+  <xacro:property name="rouder_lift_coefficient" value="171.135"/>
+  <xacro:property name="rouder_drag_coefficient" value="1.98"/>
+  <xacro:macro name="rouder_macro" params="namespace fin_id *origin mesh_filename">
       <xacro:fin_quadratic_macro
         namespace="${namespace}"
@@ -128,6 +117,6 @@
         mesh_filename="${mesh_filename}"
         fin_dynamics_time_constant="0.2"
-        lift_constant="${0.5 * fin_rho * aft_fin_area * aft_fin_lift_coefficient}"
-        drag_constant="${0.5 * fin_rho * aft_fin_area * aft_fin_drag_coefficient}"
+        lift_constant="${0.5 * fin_rho * rouder_area * rouder_lift_coefficient}"
+        drag_constant="${0.5 * fin_rho * rouder_area * rouder_drag_coefficient}"
         current_velocity_topic="current_velocity">
         <xacro:insert_block name="origin"/>

Commit message: update

File: armsauv_description/urdf/actuators.xacro (robot description, xacro)
@@ -13,11 +13,11 @@
     <!-- Instantiate fins, if necessary -->
     <xacro:fin_macro namespace="${namespace}" fin_id="0" mesh_filename="${front_fin_mesh_file}">
-      <origin xyz="1.865 -0.699 0.013" rpy="${0.5 * pi} 0 0" />
+      <origin xyz="1.865 -0.699 -0.013" rpy="${0.5 * pi} 0 0" />
     </xacro:fin_macro>
     <xacro:fin_macro namespace="${namespace}" fin_id="1" mesh_filename="${front_fin_mesh_file}">
-      <origin xyz="1.865 0.699 -0.287" rpy="${1.5 * pi} 0 0" />
+      <origin xyz="1.865 0.699 -0.013" rpy="${1.5 * pi} 0 0" />
     </xacro:fin_macro>
     <xacro:fin_macro namespace="${namespace}" fin_id="2" mesh_filename="${aft_fin_mesh_file}">
-      <origin xyz="-3.369 0.621 -0.1896" rpy="${0.5 * pi} 0 0" />
+      <origin xyz="-3.369 -0.621 0.0844" rpy="${0.5 * pi} 0 0" />
     </xacro:fin_macro>
     <xacro:rouder_macro namespace="${namespace}" fin_id="3" mesh_filename="${aft_fin_mesh_file}">
@@ -25,5 +25,5 @@
     </xacro:rouder_macro>
     <xacro:fin_macro namespace="${namespace}" fin_id="4" mesh_filename="${aft_fin_mesh_file}">
-      <origin xyz="-3.369 -0.621 -0.0844" rpy="${1.5 * pi} 0 0" />
+      <origin xyz="-3.369 0.621 0.0844" rpy="${1.5 * pi} 0 0" />
     </xacro:fin_macro>
     <xacro:rouder_macro namespace="${namespace}" fin_id="5" mesh_filename="${aft_fin_mesh_file}">

File: armsauv_description/urdf/gazebo.xacro (robot description, xacro)
@@ -2,6 +2,6 @@
 <robot xmlns:xacro="http://www.ros.org/wiki/xacro">
     <!-- Center of buoyancy -->
-    <!-- <xacro:property name="armsauv_cob" value="0.086 0 -0.137"/> -->
-    <xacro:property name="armsauv_cob" value="0.086 0 -0.137"/>
+    <xacro:property name="armsauv_cob" value="0 0 0.137"/>
+    <!-- <xacro:property name="armsauv_cob" value="0 0 0"/> -->
     <!-- Vehicle's actual volume (Gazebo cannot compute the volume out of the mesh) -->
     <!-- <xacro:property name="armsauv_volume" value="${4605 / 1025}"/> -->
@@ -13,4 +13,5 @@
     <xacro:property name="armsauv_radius"  value="0.35795"/>
     <xacro:property name="armsauv_height" value="1.4318"/>
+    <xacro:property name="factor" value="0.65"/>
     <xacro:macro name="armsauv_hydro_model" params="namespace">
       <!-- List of hydrodynamic models this robot's links -->
@@ -34,10 +35,10 @@
           <type>fossen</type>
           <added_mass>
-            1.432   0       0       0     0      0
+            <!-- 1.432   0       0       0     0      0
             0    120.645    0       0     0    4.895
             0       0    130.513    0  -16.488   0
             0       0       0    0.386    0      0
             0       0   -16.488     0  78.266    0
-            0     4.895     0       0     0    67.489
+            0     4.895     0       0     0    67.489 -->
             <!-- 302.286     0         0          0          0           0
             0       12996.067     0          0          0        3778.498
@@ -53,15 +54,15 @@
             0           0         0          0         0        42452.977 -->
             <!-- 302.286     0        0          0          0          0
-            0       12996.067    0       1486.934      0        3778.498
-            0           0     7198.801      0      -138.636       0
-            0        1486.934    0      2435.827       0       -85.834
-            0           0    -138.636       0       40597.109     0
-            0        3778.498    0       -85.834       0        42452.977 -->
-            <!-- 30.2285     0         0          0         0           0
-            0       1299.6067     0      -148.6934     0      -377.8498
-            0           0     719.8802       0       13.8636       0
-            0       -148.6934     0       243.5827     0        8.5834
-            0           0     13.8636        0      4059.7109      0
-            0       -377.8498     0        8.5834      0       4245.2977 -->
+            0       12996.067    0      -1486.934      0       -3778.498
+            0           0     7198.801      0       138.636       0
+            0       -1486.934    0       2435.827      0        85.834
+            0           0     138.636       0       40597.109     0
+            0       -3778.498    0        85.834       0        42452.977 -->
+  ${302.285 * factor}         0               0               0               0               0
+            0     ${12996.067 * factor}       0    ${-1486.934 * factor}      0       ${-3778.498 * factor}
+            0                 0     ${7198.802 * factor}      0       ${138.636 * factor}      0
+            0       ${-1486.934 * factor}     0     ${2435.827 * factor}      0         ${85.834 * factor}
+            0                 0     ${138.636 * factor}       0      ${40597.109 * factor}     0
+            0       ${-3778.498 * factor}     0    ${85.834 * factor}         0       ${42452.977 * factor}
             <!-- 302.285     0         0          0         0           0
             0       12996.067     0          0         0           0

File: armsauv_description/urdf/snippets.xacro (robot description, xacro)
@@ -87,6 +87,6 @@
   <!-- Fin properties -->
   <xacro:property name="fin_rho" value="1025"/>
-  <xacro:property name="fin_area" value="1"/>
-  <xacro:property name="fin_lift_coefficient" value="373.249"/>
+  <xacro:property name="fin_area" value="0.0400"/>
+  <xacro:property name="fin_lift_coefficient" value="${ 373.249 * 2 / fin_rho / fin_area}"/>
   <xacro:property name="fin_drag_coefficient" value="1.98"/>
   <xacro:macro name="fin_macro" params="namespace fin_id *origin mesh_filename">
@@ -105,6 +105,6 @@
       </xacro:fin_quadratic_macro>
   </xacro:macro>
-  <xacro:property name="rouder_area" value="1"/>
-  <xacro:property name="rouder_lift_coefficient" value="171.135"/>
+  <xacro:property name="rouder_area" value="0.0541"/>
+  <xacro:property name="rouder_lift_coefficient" value="${ 171.135 * 2 / fin_rho / rouder_area }"/>
   <xacro:property name="rouder_drag_coefficient" value="1.98"/>
   <xacro:macro name="rouder_macro" params="namespace fin_id *origin mesh_filename">
