Commit message: Add camera plugin

File: armsauv_description/urdf/sensors.xacro (robot description, xacro)
@@ -4,8 +4,81 @@
   <xacro:default_gps namespace="${namespace}" parent_link="${namespace}/base_link" />
   <!-- Mount a Pose 3D sensor. -->
-  <xacro:default_pose_3d_macro
+  <!-- <xacro:default_pose_3d_macro
     namespace="${namespace}"
     parent_link="${namespace}/base_link"
-    inertial_reference_frame="${inertial_reference_frame}" />
+    inertial_reference_frame="${inertial_reference_frame}" /> -->
+  <xacro:pose_3d_macro
+      	  namespace="${namespace}"
+      	  parent_link="${namespace}/base_link"
+      	  topic="pose_gt"
+      	  update_rate="10"
+      	  noise_sigma="0.0"
+      	  noise_amplitude="0.0"
+      	  suffix="default"
+      	  reference_frame="world"
+      	  publish_ned_odom="false">
+    <origin xyz="0 0 0" rpy="0 0 0"/>
+  </xacro:pose_3d_macro>
+  <xacro:macro name="arms_camera" params="namespace">
+    <!-- Monocular Camera -->
+    <link name="${namespace}">
+      <visual>
+        <origin xyz="1.35 0 0.03" rpy="0 0 0.78539164"/>
+      </visual>
+      <collision>
+        <origin xyz="1.35 0 0.03" rpy="0 0 0.78539164"/>
+        <geometry>
+          <cylinder radius="0.015" length="0.042" />
+        </geometry>
+        <inertial>
+          <mass value="0.3" />
+          <inertia
+            ixx="0.0000450"
+            iyy="0.0001746"
+            izz="0.0001746"
+            ixy="0"
+            ixz="0"
+            iyz="0"/>
+        </inertial>
+      </collision>
+    </link>
+    <!-- Gazebo camera setup -->
+    <gazebo reference="${namespace}/base_link">
+      <sensor type="camera" name="${namespace}/sensor">
+        <update_rate>10.0</update_rate>
+        <camera name="camera">
+          <horizontal_fov>1.3962634</horizontal_fov>
+          <image>
+            <width>1280</width>
+            <height>720</height>
+            <format>R8GB8</format>
+          </image>
+          <clip>
+            <near>0.05</near>
+            <far>10</far>
+          </clip>
+          <noise>
+            <type>gaussian</type>
+            <mean>0.0</mean>
+            <stddev>0.007</stddev>
+          </noise>
+        </camera>
+        <plugin name="camera_plugin" filename="libgazebo_ros_camera.so">
+          <alwaysOn>true</alwaysOn>
+          <updateRate>0.0</updateRate>
+          <cameraName>${namespace}/${sensor_namespace}/${camera_namespace}</cameraName>
+          <imageTopicName>image_raw</imageTopicName>
+          <cameraInfoTopicName>camera_info</cameraInfoTopicName>
+          <frameName>${namespace}/base_link</frameName>
+          <hackBaseline></hackBaseline>
+          <distortionK1>0.0</distortionK1>
+          <distortionK2>0.0</distortionK2>
+          <distortionK3>0.0</distortionK3>
+          <distortionT1>0.0</distortionT1>
+          <distortionT2>0.0</distortionT2>
+        </plugin>
+      </sensor>
+    </gazebo>
+  </xacro:macro>
   <xacro:macro name="arms_forward_multibeam_p900" params="namespace parent_link *origin">
     <xacro:multibeam_sonar

Commit message: Remove uuv camera plugin and multibeam sonar plugin

File: armsauv_description/urdf/sensors.xacro (robot description, xacro)
@@ -3,9 +3,5 @@
   <!-- Mount a GPS. -->
   <xacro:default_gps namespace="${namespace}" parent_link="${namespace}/base_link" />
-  <!-- Mount a Pose 3D sensor. -->
-  <!-- <xacro:default_pose_3d_macro
-    namespace="${namespace}"
-    parent_link="${namespace}/base_link"
-    inertial_reference_frame="${inertial_reference_frame}" /> -->
+  <!-- Mount a Virtual Pose Sensor-->
   <xacro:pose_3d_macro
       	  namespace="${namespace}"
@@ -15,106 +11,19 @@
       	  noise_sigma="0.0"
       	  noise_amplitude="0.0"
-      	  suffix="default"
+      	  suffix=""
       	  reference_frame="world"
       	  publish_ned_odom="false">
     <origin xyz="0 0 0" rpy="0 0 0"/>
   </xacro:pose_3d_macro>
-  <xacro:macro name="arms_camera" params="namespace">
-    <!-- Monocular Camera -->
-    <link name="${namespace}">
-      <visual>
-        <origin xyz="1.35 0 0.03" rpy="0 0 0.78539164"/>
-      </visual>
-      <collision>
-        <origin xyz="1.35 0 0.03" rpy="0 0 0.78539164"/>
-        <geometry>
-          <cylinder radius="0.015" length="0.042" />
-        </geometry>
-        <inertial>
-          <mass value="0.3" />
-          <inertia
-            ixx="0.0000450"
-            iyy="0.0001746"
-            izz="0.0001746"
-            ixy="0"
-            ixz="0"
-            iyz="0"/>
-        </inertial>
-      </collision>
-    </link>
-    <!-- Gazebo camera setup -->
-    <gazebo reference="${namespace}/base_link">
-      <sensor type="camera" name="${namespace}/sensor">
-        <update_rate>10.0</update_rate>
-        <camera name="camera">
-          <horizontal_fov>1.3962634</horizontal_fov>
-          <image>
-            <width>1280</width>
-            <height>720</height>
-            <format>R8GB8</format>
-          </image>
-          <clip>
-            <near>0.05</near>
-            <far>10</far>
-          </clip>
-          <noise>
-            <type>gaussian</type>
-            <mean>0.0</mean>
-            <stddev>0.007</stddev>
-          </noise>
-        </camera>
-        <plugin name="camera_plugin" filename="libgazebo_ros_camera.so">
-          <alwaysOn>true</alwaysOn>
-          <updateRate>0.0</updateRate>
-          <cameraName>${namespace}/${sensor_namespace}/${camera_namespace}</cameraName>
-          <imageTopicName>image_raw</imageTopicName>
-          <cameraInfoTopicName>camera_info</cameraInfoTopicName>
-          <frameName>${namespace}/base_link</frameName>
-          <hackBaseline></hackBaseline>
-          <distortionK1>0.0</distortionK1>
-          <distortionK2>0.0</distortionK2>
-          <distortionK3>0.0</distortionK3>
-          <distortionT1>0.0</distortionT1>
-          <distortionT2>0.0</distortionT2>
-        </plugin>
-      </sensor>
-    </gazebo>
-  </xacro:macro>
-  <xacro:macro name="arms_forward_multibeam_p900" params="namespace parent_link *origin">
-    <xacro:multibeam_sonar
-      namespace="${namespace}"
-      suffix=""
-      parent_link="${parent_link}"
-      topic="sonar"
-      mass="0.001"
-      update_rate="15"
-      samples="512"
-      fov="1.5708"
-      range_min="1.0"
-      range_max="100.0"
-      range_stddev="0.027"
-      mesh="">
-      <inertia ixx="0.0" ixy="0.0" ixz="0.0" iyy="0.0" iyz="0.0" izz="0.0" />
-      <xacro:insert_block name="origin" />
-      <visual>
-        <geometry>
-          <mesh filename="file://$(find uuv_sensor_ros_plugins)/meshes/p900.dae" scale="1 1 1"/>
-        </geometry>
-      </visual>
-    </xacro:multibeam_sonar>
-  </xacro:macro>
-  <!-- Forward-looking sonar sensor -->
-  <xacro:arms_forward_multibeam_p900 namespace="${namespace}" parent_link="${namespace}/base_link">
-    <origin xyz="0 0 0" rpy="0 0 0"/>
-  </xacro:arms_forward_multibeam_p900>
   <!-- DVL  -->
   <xacro:default_dvl namespace="${namespace}" parent_link="${namespace}/base_link">
     <origin xyz="0 0 0" rpy="0 0 0"/>
   </xacro:default_dvl>
-  <xacro:macro name="arms_pressure" params="namespace parent_link *origin">
+  <!-- Mount a Pressure Sensor -->
+  <xacro:macro name="arms_pressure" params="namespace">
     <xacro:pressure_plugin_macro
       namespace="${namespace}"
       suffix=""
-      parent_link="${parent_link}"
+      parent_link="${namespace}/base_link"
       topic="pressure"
       mass="0.001"
@@ -127,17 +36,14 @@
       kPaPerM="9.80638">
       <inertia ixx="0.0" ixy="0.0" ixz="0.0" iyy="0.0" iyz="0.0" izz="0.0" />
-      <xacro:insert_block name="origin" />
+      <origin xyz="0 0 0" rpy="0 0 0"/>
     </xacro:pressure_plugin_macro>
   </xacro:macro>
-  <!-- Pressure  -->
-  <xacro:arms_pressure namespace="${namespace}" parent_link="${namespace}/base_link">
-    <origin xyz="0 0 0" rpy="0 0 0"/>
-  </xacro:arms_pressure>
-  <xacro:macro name="arms_imu" params="namespace parent_link *origin">
+  <!-- Mount an IMU -->
+  <xacro:macro name="arms_imu" params="namespace">
     <!-- ADIS16448 IMU. -->
     <xacro:imu_plugin_macro
       namespace="${namespace}"
       imu_suffix=""
-      parent_link="${parent_link}"
+      parent_link="${namespace}/base_link"
       imu_topic="imu"
       mass_imu_sensor="0.001"
@@ -155,11 +61,7 @@
       update_rate="50">
       <inertia ixx="0.0" ixy="0.0" ixz="0.0" iyy="0.0" iyz="0.0" izz="0.0" />
-      <xacro:insert_block name="origin" />
+      <origin xyz="0 0 0" rpy="0 0 0"/>
     </xacro:imu_plugin_macro>
   </xacro:macro>
-  <!-- IMU  -->
-  <xacro:arms_imu namespace="${namespace}" parent_link="${namespace}/base_link">
-    <origin xyz="0 0 0" rpy="0 0 0"/>
-  </xacro:arms_imu>
   <!-- Mount the chemical concentration sensor -->
   <xacro:chemical_concentration_sensor_macro

Commit message: Remove default multibeam sonar

File: armsauv_description/urdf/sensors.xacro (robot description, xacro)
@@ -16,4 +16,27 @@
     <origin xyz="0 0 0" rpy="0 0 0"/>
   </xacro:pose_3d_macro>
+  <!--<xacro:macro name="forward_multibeam_p900" params="namespace">
+    <xacro:multibeam_sonar
+      namespace="${namespace}"
+      suffix=""
+      parent_link="${namespace}/base_link"
+      topic="forward_multibeam"
+      mass="0.02"
+      update_rate="15"
+      samples="512"
+      fov="1.5708"
+      range_min="1.0"
+      range_max="100.0"
+      range_stddev="0.027"
+      mesh="">
+      <inertia ixx="0.00001" ixy="0.0" ixz="0.0" iyy="0.00001" iyz="0.0" izz="0.00001" />
+      <origin xyz="0.75 0 -0.3" rpy="0 0 0"/>
+      <visual>
+        <geometry>
+          <mesh filename="file://$(find uuv_sensor_ros_plugins)/meshes/p900.dae" scale="0.5 0.5 0.5"/>
+        </geometry>
+      </visual>
+    </xacro:multibeam_sonar>
+  </xacro:macro>-->
   <!-- DVL  -->
   <xacro:default_dvl namespace="${namespace}" parent_link="${namespace}/base_link">
