Commit message: fix mass and volume

File: armsauv_description/urdf/base.xacro (robot description, xacro)
@@ -12,5 +12,5 @@
     Vehicle's parameters (remember to enter the model parameters below)
   -->
-  <xacro:property name="mass" value="831"/>
+  <xacro:property name="mass" value="${831 / 9.8}"/>
   <!-- Center of gravity -->
   <xacro:property name="cog" value="0 0 0.0086"/>
@@ -50,5 +50,5 @@
         </visual>
         <collision>
-          <origin xyz="0 0 0" rpy="0 0 0"/>s
+          <origin xyz="-0.5 0 0" rpy="0 0 0"/>s
           <geometry>
             <mesh filename="${collision_mesh_file}" scale="1 1 1" />

File: armsauv_description/urdf/gazebo.xacro (robot description, xacro)
@@ -4,5 +4,5 @@
     <xacro:property name="armsauv_cob" value="0 0 0"/>
     <!-- Vehicle's actual volume (Gazebo cannot compute the volume out of the mesh) -->
-    <xacro:property name="armsauv_volume" value="0.838"/>
+    <xacro:property name="armsauv_volume" value="${838 / 9.8 / 1000}"/>
     <!-- Describing the dimensions of the vehicle's bounding box -->
     <xacro:property name="armsauv_length" value="2.712"/>

File: armsauv_description/urdf/snippets.xacro (robot description, xacro)
@@ -49,7 +49,7 @@
         <gain>1</gain>
         <!-- Maximum allowed input value for the input signal for thruster unit -->
-        <clampMax>-3000</clampMax>
+        <clampMax>3000</clampMax>
         <!-- Minimum allowed value for the input signal for thruster unit -->
-        <clampMin>3000</clampMin>
+        <clampMin>-3000</clampMin>
         <!-- Minimum and maximum thrust force output allowed -->
         <thrustMin>-50</thrustMin>

Commit message: Add gazebo camera link and joint

File: armsauv_description/urdf/base.xacro (robot description, xacro)
@@ -30,30 +30,170 @@
   <!-- Vehicle macro -->
   <xacro:macro name="armsauv_base" params="namespace *gazebo inertial_reference_frame">
-      <!-- Rigid body description of the base link -->
-      <link name="${namespace}/base_link">
-        <!--
-          Be careful to setup the coefficients for the inertial tensor,
-          otherwise your model will become unstable on Gazebo
-        -->
-        <inertial>
-          <mass value="${mass}" />
-          <origin xyz="${cog}" rpy="0 0 0"/>
-          <inertia ixx="0.82" ixy="0" ixz="0"
-                   iyy="30.14" iyz="0"
-                   izz="30.14" />
-        </inertial>
-        <visual>
-          <origin xyz="-0.5 0 0" rpy="0 0 0"/>
-          <geometry>
-            <mesh filename="${visual_mesh_file}" scale="1 1 1" />
-          </geometry>
-        </visual>
-        <collision>
-          <origin xyz="-0.5 0 0" rpy="0 0 0"/>s
-          <geometry>
-            <mesh filename="${collision_mesh_file}" scale="1 1 1" />
-          </geometry>
-        </collision>
-      </link>
+    <!-- Rigid body description of the base link -->
+    <link name="${namespace}/base_link">
+      <!--
+        Be careful to setup the coefficients for the inertial tensor,
+        otherwise your model will become unstable on Gazebo
+      -->
+      <inertial>
+        <mass value="${mass}" />
+        <origin xyz="${cog}" rpy="0 0 0"/>
+        <inertia ixx="0.82" ixy="0" ixz="0"
+                 iyy="30.14" iyz="0"
+                 izz="30.14" />
+      </inertial>
+      <visual>
+        <origin xyz="-0.5 0 0" rpy="0 0 0"/>
+        <geometry>
+          <mesh filename="${visual_mesh_file}" scale="1 1 1" />
+        </geometry>
+      </visual>
+      <collision>
+        <origin xyz="-0.5 0 0" rpy="0 0 0"/>
+        <geometry>
+          <mesh filename="${collision_mesh_file}" scale="1 1 1" />
+        </geometry>
+      </collision>
+    </link>
+    <link name="${namespace}/camera_link">
+      <mass value="0.3"/>
+      <origin xyz="0 0 0" rpy="0 0 0"/>
+      <inertia
+          ixx="0.0000450"
+          iyy="0.0001746"
+          izz="0.0001746"
+          ixy="0"
+          ixz="0"
+          iyz="0"/>
+      <visual>
+        <origin xyz="0 0 0" rpy="0 0 1.57"/>
+        <geometry>
+          <mesh filename="file://$(find armsauv_description)/meshes/sensors/mono_camera/mesh/mono_camera.dae" scale="1 1 1"/>
+        </geometry>
+      </visual>
+      <collision>
+        <origin xyz="0 0 0" rpy="0 0 1.57"/>
+        <geometry>
+          <mesh filename="file://$(find armsauv_description)/meshes/sensors/mono_camera/mesh/mono_camera.dae" scale="1 1 1"/>
+        </geometry>
+      </collision>
+    </link>
+    <joint name="${namespace}/camera_to_base" type="fixed">
+      <parent link ="${namespace}/base_link"/>
+      <child link ="${namespace}/camera_link"/>
+      <origin rpy="0 0 0" xyz="0.85 0 0"/>
+      <axis xyz="1 0 0"/>
+    </joint>
+    <link name="${namespace}/multibeam_sonar_link" type="fixed">
+      <mass value="0.02"/>
+      <origin xyz="0 0 0" rpy="0 0 0"/>
+      <inertia
+          ixx="0.00001"
+          iyy="0.00001"
+          izz="0.00001"
+          ixy="0.0"
+          ixz="0.0"
+          iyz="0.0"/>
+      <visual>
+        <origin xyz="0 0 0" rpy="0 0 0"/>
+        <geometry>
+          <mesh filename="file://$(find uuv_sensor_ros_plugins)/meshes/p900.dae" scale="1 1 1"/>
+        </geometry>
+      </visual>
+      <collision>
+        <origin xyz="0 0 0" rpy="0 0 0"/>
+        <geometry>
+          <mesh filename="file://$(find uuv_sensor_ros_plugins)/meshes/p900.dae" scale="1 1 1"/>
+        </geometry>
+      </collision>
+    </link>
+    <joint name="multibeam_to_base" type="fixed">
+      <parent link="${namespace}/base_link"/>
+      <child link="${namespace}/multibeam_sonar_link" />
+      <origin rpy="0 0 0" xyz="0.75 0 -0.3"/>
+      <axis xyz="1 0 0"/>
+    </joint>
+    <gazebo reference="${namespace}/camera_link">
+      <sensor type="camera" name="sensor">
+        <update_rate>10.0</update_rate>
+        <camera name="camera">
+          <horizontal_fov>1.3962634</horizontal_fov>
+          <image>
+            <width>1280</width>
+            <height>720</height>
+            <format>R8G8B8</format>
+          </image>
+          <clip>
+            <near>0.05</near>
+            <far>10</far>
+          </clip>
+          <noise>
+            <type>gaussian</type>
+            <mean>0.0</mean>
+            <stddev>0.007</stddev>
+          </noise>
+        </camera>
+	<!--<plugin name="camera_plugin" filename="libuuv_gazebo_ros_camera_plugin.so">
+          <updateRate>10.0</updateRate>
+          <cameraName>camera</cameraName>
+	  <frameName>${namespace}/camera_link</frameName>
+	  <attenuationR>0.01</attenuationR>
+	  <attenuationG>0.03</attenuationG>
+	  <attenuationB>0.01</attenuationB>
+	  <backgroundR>0</backgroundR>
+	  <backgroundG>0</backgroundG>
+	  <backgroundB>0</backgroundB>
+	  <imageTopicName>image</imageTopicName>
+	  <pointCloudTopicName>cloud_point</pointCloudTopicName>
+	  <depthImageTopicName>depth</depthImageTopicName>
+	  <depthImageCameraInfoTopicName>depth_info</depthImageCameraInfoTopicName>
+	  <pointCloudCutoff>10.0</pointCloudCutoff>
+	</plugin>-->
+	<plugin name="camera_plugin" filename="libgazebo_ros_camera.so">
+          <alwaysOn>true</alwaysOn>
+          <updateRate>10.0</updateRate>
+          <cameraName>camera</cameraName>
+          <frameName>camera_link</frameName>
+          <hackBaseline>0.07</hackBaseline>
+          <distortionK1>0.0</distortionK1>
+          <distortionK2>0.0</distortionK2>
+          <distortionK3>0.0</distortionK3>
+          <distortionT1>0.0</distortionT1>
+          <distortionT2>0.0</distortionT2>
+          <imageTopicName>image</imageTopicName>
+          <cameraInfoTopicName>camera_info</cameraInfoTopicName>
+        </plugin>
+      </sensor>
+    </gazebo>
+    <gazebo reference="${namespace}/multibeam_sonar_link">
+      <sensor type="gpu_ray" name="multibeam_sonar">
+        <visualize>false</visualize>
+        <update_rate>10.0</update_rate>
+        <ray>
+          <scan>
+            <horizontal>
+              <samples>500</samples>
+              <resolution>0.1</resolution>
+              <min_angle>-0.785398163</min_angle><!--45-->
+              <max_angle>0.785398163</max_angle><!--45-->
+            </horizontal>
+          </scan>
+          <range>
+            <min>1</min>
+            <max>60</max>
+            <resolution>0.01</resolution>
+          </range>
+          <noise>
+            <type>gaussian</type>
+            <mean>0.0</mean>
+            <stddev>0.001</stddev>
+          </noise>
+        </ray>
+        <plugin name="multibeam_sonar_plugin" filename="libgazebo_ros_gpu_laser.so">
+          <topicName>multibeam_sonar_image</topicName>
+          <frameName>multibeam_sonar_link</frameName>
+        </plugin>
+      </sensor>
+    </gazebo>
     <gazebo reference="${namespace}/base_link">
       <selfCollide>false</selfCollide>

Commit message: Add multibeam sonar

File: armsauv_description/urdf/base.xacro (robot description, xacro)
@@ -98,5 +98,5 @@
         <origin xyz="0 0 0" rpy="0 0 0"/>
         <geometry>
-          <mesh filename="file://$(find uuv_sensor_ros_plugins)/meshes/p900.dae" scale="1 1 1"/>
+          <mesh filename="file://$(find uuv_sensor_ros_plugins)/meshes/p900.dae" scale="0.5 0.5 0.5"/>
         </geometry>
       </visual>
@@ -104,5 +104,5 @@
         <origin xyz="0 0 0" rpy="0 0 0"/>
         <geometry>
-          <mesh filename="file://$(find uuv_sensor_ros_plugins)/meshes/p900.dae" scale="1 1 1"/>
+          <mesh filename="file://$(find uuv_sensor_ros_plugins)/meshes/p900.dae" scale="0.5 0.5 0.5"/>
         </geometry>
       </collision>
@@ -168,19 +168,19 @@
     <gazebo reference="${namespace}/multibeam_sonar_link">
       <sensor type="gpu_ray" name="multibeam_sonar">
-        <visualize>false</visualize>
-        <update_rate>10.0</update_rate>
+        <visualize>true</visualize>
+        <update_rate>15.0</update_rate>
         <ray>
           <scan>
             <horizontal>
-              <samples>500</samples>
-              <resolution>0.1</resolution>
-              <min_angle>-0.785398163</min_angle><!--45-->
-              <max_angle>0.785398163</max_angle><!--45-->
+              <samples>512</samples>
+              <resolution>0.01</resolution>
+              <min_angle>-0.785398163</min_angle>
+              <max_angle>0.785398163</max_angle>
             </horizontal>
           </scan>
           <range>
-            <min>1</min>
+            <min>2</min>
             <max>60</max>
-            <resolution>0.01</resolution>
+            <resolution>1</resolution>
           </range>
           <noise>
@@ -191,5 +191,5 @@
         </ray>
         <plugin name="multibeam_sonar_plugin" filename="libgazebo_ros_gpu_laser.so">
-          <topicName>multibeam_sonar_image</topicName>
+          <topicName>multibeam_sonar</topicName>
           <frameName>multibeam_sonar_link</frameName>
         </plugin>

Commit message: Update link of forward looking sonar

File: armsauv_description/urdf/base.xacro (robot description, xacro)
@@ -85,5 +85,5 @@
       <axis xyz="1 0 0"/>
     </joint>
-    <link name="${namespace}/multibeam_sonar_link" type="fixed">
+    <!--<link name="${namespace}/multibeam_sonar_link" type="fixed">
       <mass value="0.02"/>
       <origin xyz="0 0 0" rpy="0 0 0"/>
@@ -112,4 +112,33 @@
       <child link="${namespace}/multibeam_sonar_link" />
       <origin rpy="0 0 0" xyz="0.75 0 -0.3"/>
+      <axis xyz="1 0 0"/>
+    </joint>-->
+    <link name="${namespace}/forward_looking_sonar_link" type="fixed">
+      <mass value="0.02"/>
+      <origin xyz="0 0 0" rpy="0 0 0"/>
+      <inertia
+          ixx="0.00001"
+          iyy="0.00001"
+          izz="0.00001"
+          ixy="0.0"
+          ixz="0.0"
+          iyz="0.0"/>
+      <visual>
+        <origin xyz="0 0 0" rpy="0 0 0"/>
+        <geometry>
+          <mesh filename="file://$(find uuv_sensor_ros_plugins)/meshes/oe14-372.dae" scale="0.5 0.5 0.5"/>
+        </geometry>
+      </visual>
+      <collision>
+        <origin xyz="0 0 0" rpy="0 0 0"/>
+        <geometry>
+          <mesh filename="file://$(find uuv_sensor_ros_plugins)/meshes/oe14-372.dae" scale="0.5 0.5 0.5"/>
+        </geometry>
+      </collision>
+    </link>
+    <joint name="forwardlooking_to_base" type="fixed">
+      <parent link="${namespace}/base_link"/>
+      <child link="${namespace}/forward_looking_sonar_link" />
+      <origin rpy="0 0 0" xyz="0.75 0 -0.125"/>
       <axis xyz="1 0 0"/>
     </joint>
@@ -166,5 +195,5 @@
       </sensor>
     </gazebo>
-    <gazebo reference="${namespace}/multibeam_sonar_link">
+    <!--<gazebo reference="${namespace}/multibeam_sonar_link">
       <sensor type="gpu_ray" name="multibeam_sonar">
         <visualize>true</visualize>
@@ -195,4 +224,27 @@
         </plugin>
       </sensor>
+    </gazebo>-->
+    <gazebo reference="${namespace}/forward_looking_sonar_link">
+      <sensor name="${namespace}/image_sonar" type="depth">
+        <camera>
+          <horizontal_fov>1.57</horizontal_fov>
+          <image>
+            <width>1280</width>
+            <height>720</height>
+            <format>R8G8B8</format>
+          </image>
+          <clip>
+            <save enable="true">
+              <path>/tmp/camera</path>
+            </save>
+          </clip>
+        </camera>
+        <plugin filename="libimage_sonar_ros_plugin.so" name="forward_looking_sonar">
+          <topicName>forward_looking_sonar</topicName>
+          <frameName>forward_looking_sonar_link"</frameName>
+        </plugin>
+        <alwaysOn>true</alwaysOn>
+        <update_rate>10.0</update_rate>
+      </sensor>
     </gazebo>
     <gazebo reference="${namespace}/base_link">

Commit message: Add led group

File: armsauv_description/urdf/base.xacro (robot description, xacro)
@@ -114,5 +114,5 @@
       <axis xyz="1 0 0"/>
     </joint>-->
-    <link name="${namespace}/forward_looking_sonar_link" type="fixed">
+    <link name="${namespace}/forward_looking_sonar_link">
       <mass value="0.02"/>
       <origin xyz="0 0 0" rpy="0 0 0"/>
@@ -143,4 +143,195 @@
       <axis xyz="1 0 0"/>
     </joint>
+    <link name="${namespace}/led0_link">
+      <mass value="0.1"/>
+      <origin xyz="0 0 0" rpy="0 0 0"/>
+      <inertia
+          ixx="0.00001"
+          iyy="0.00001"
+          izz="0.00001"
+          ixy="0.0"
+          ixz="0.0"
+          iyz="0.0"/>
+      <visual>
+        <origin xyz="0 0 0" rpy="0 0 0"/>
+        <geometry>
+          <box size="0.2 0.04 0.01"/>
+        </geometry>
+        <material name="lblue">
+          <color rgba="0.5294 0.8078 0.9804 1"/>
+        </material>
+      </visual>
+      <collision>
+        <origin xyz="0 0 0" rpy="0 0 0"/>
+        <geometry>
+          <box size="0.2 0.04 0.01"/>
+        </geometry>
+      </collision>
+      <!--<light name="led1" type="spot">
+        <attenuation>
+          <range>30.0</range>
+          <linear>0.05</linear>
+        </attenuation>
+        <diffuse>1 0 0 1</diffuse>
+        <specular>1 0 0 1</specular>
+        <spot>
+          <inner_angle>0.3</inner_angle>
+          <outer_angle>0.35</outer_angle>
+          <falloff>1</falloff>
+        </spot>
+        <direction>0 0 -1</direction>
+      </light>-->
+    </link>
+    <joint name="led0_to_base" type="fixed">
+      <parent link="${namespace}/base_link"/>
+      <child link="${namespace}/led0_link"/>
+      <origin xyz="-0.5 0.0 -0.12" rqy="0 0 0"/>
+      <axis xyz="0 0 1"/>
+    </joint>
+    <gazebo reference="${namespace}/led0_link">
+      <!--<light name="${namespace}/led0_link/led0" type="spot">-->
+      <light name="${namespace}/led0_link/led0" type="directional">
+        <pose>-0.5 0.0 -0.12 0 0 0</pose>
+        <attenuation>
+          <range>5.0</range>
+          <linear>0.05</linear>
+        </attenuation>
+        <diffuse>1 0 0 1</diffuse>
+        <specular>1 0 0 1</specular>
+        <!--<spot>
+          <inner_angle>0.3</inner_angle>
+          <outer_angle>0.35</outer_angle>
+          <falloff>1</falloff>
+        </spot>-->
+        <direction>0 0 -1</direction>
+      </light>
+      <plugin name="led_control" filename="libFlashLightPlugin.so">
+        <enable>true</enable>
+        <light>
+          <id>${namespace}/led0_link/led0</id>
+          <duration>1.0</duration>
+          <interval>0</interval>
+          <color>1 0 0</color>
+        </light>
+      </plugin>
+    </gazebo>
+    <link name="${namespace}/led1_link">
+      <mass value="0.1"/>
+      <origin xyz="0 0 0" rpy="0 0 0"/>
+      <inertia
+          ixx="0.00001"
+          iyy="0.00001"
+          izz="0.00001"
+          ixy="0.0"
+          ixz="0.0"
+          iyz="0.0"/>
+      <visual>
+        <origin xyz="0 0 0" rpy="0 0 0"/>
+        <geometry>
+          <box size="0.2 0.04 0.01"/>
+        </geometry>
+        <material name="lblue">
+          <color rgba="0.5294 0.8078 0.9804 1"/>
+        </material>
+      </visual>
+      <collision>
+        <origin xyz="0 0 0" rpy="0 0 0"/>
+        <geometry>
+          <box size="0.2 0.04 0.01"/>
+        </geometry>
+      </collision>
+    </link>
+    <joint name="led1_to_base" type="fixed">
+      <parent link="${namespace}/base_link"/>
+      <child link="${namespace}/led1_link"/>
+      <origin xyz="-0.29 0.0 -0.12" rqy="0 0 0"/>
+      <axis xyz="0 0 1"/>
+    </joint>
+    <gazebo reference="${namespace}/led1_link">
+      <!--<light name="${namespace}/led1_link/led1" type="spot">-->
+      <light name="${namespace}/led1_link/led1" type="directional">
+        <pose>-0.29 0.0 -0.12 0 0 0</pose>
+        <attenuation>
+          <range>5.0</range>
+          <linear>0.05</linear>
+        </attenuation>
+        <diffuse>1 0 0 1</diffuse>
+        <specular>1 0 0 1</specular>
+        <!--<spot>
+          <inner_angle>0.3</inner_angle>
+          <outer_angle>0.35</outer_angle>
+          <falloff>1</falloff>
+        </spot>-->
+        <direction>0 0 -1</direction>
+      </light>
+      <plugin name="led_control" filename="libFlashLightPlugin.so">
+        <enable>true</enable>
+        <light>
+          <id>${namespace}/led1_link/led1</id>
+          <duration>1.0</duration>
+          <interval>0</interval>
+          <color>1 0 0</color>
+        </light>
+      </plugin>
+    </gazebo>
+    <link name="${namespace}/led2_link">
+      <mass value="0.1"/>
+      <origin xyz="0 0 0" rpy="0 0 0"/>
+      <inertia
+          ixx="0.00001"
+          iyy="0.00001"
+          izz="0.00001"
+          ixy="0.0"
+          ixz="0.0"
+          iyz="0.0"/>
+      <visual>
+        <origin xyz="0 0 0" rpy="0 0 0"/>
+        <geometry>
+          <box size="0.2 0.04 0.01"/>
+        </geometry>
+        <material name="lblue">
+          <color rgba="0.5294 0.8078 0.9804 1"/>
+        </material>
+      </visual>
+      <collision>
+        <origin xyz="0 0 0" rpy="0 0 0"/>
+          <geometry>
+            <box size="0.2 0.04 0.01"/>
+          </geometry>
+      </collision>
+    </link>
+    <joint name="led2_to_base" type="fixed">
+      <parent link="${namespace}/base_link"/>
+      <child link="${namespace}/led2_link"/>
+      <origin xyz="-0.71 0.0 -0.12" rqy="0 0 0"/>
+      <axis xyz="0 0 1"/>
+    </joint>
+    <gazebo reference="${namespace}/led2_link">
+      <!--<light name="${namespace}/led2_link/led2" type="spot">-->
+      <light name="${namespace}/led2_link/led2" type="directional">
+        <pose>-0.71 0.0 -0.12 0 0 0</pose>
+        <attenuation>
+          <range>5.0</range>
+          <linear>0.05</linear>
+        </attenuation>
+        <diffuse>1 0 0 1</diffuse>
+        <specular>1 0 0 1</specular>
+        <!--<spot>
+          <inner_angle>0.3</inner_angle>
+          <outer_angle>0.35</outer_angle>
+          <falloff>1</falloff>
+        </spot>-->
+        <direction>0 0 -1</direction>
+      </light>
+      <plugin name="led_control" filename="libFlashLightPlugin.so">
+        <enable>true</enable>
+        <light>
+          <id>${namespace}/led2_link/led2</id>
+          <duration>1.0</duration>
+          <interval>0</interval>
+          <color>1 0 0</color>
+        </light>
+      </plugin>
+    </gazebo>
     <gazebo reference="${namespace}/camera_link">
       <sensor type="camera" name="sensor">

Commit message: Change mass of virtual sensors

File: armsauv_description/urdf/base.xacro (robot description, xacro)
@@ -57,5 +57,5 @@
     </link>
     <link name="${namespace}/camera_link">
-      <mass value="0.3"/>
+      <mass value="0.03"/>
       <origin xyz="0 0 0" rpy="0 0 0"/>
       <inertia
@@ -144,5 +144,5 @@
     </joint>
     <link name="${namespace}/led0_link">
-      <mass value="0.1"/>
+      <mass value="0.01"/>
       <origin xyz="0 0 0" rpy="0 0 0"/>
       <inertia
@@ -217,5 +217,5 @@
     </gazebo>
     <link name="${namespace}/led1_link">
-      <mass value="0.1"/>
+      <mass value="0.03"/>
       <origin xyz="0 0 0" rpy="0 0 0"/>
       <inertia
@@ -276,5 +276,5 @@
     </gazebo>
     <link name="${namespace}/led2_link">
-      <mass value="0.1"/>
+      <mass value="0.03"/>
       <origin xyz="0 0 0" rpy="0 0 0"/>
       <inertia
